File: pcb/yuletronics.sch (KiCad schematic (older format))
At the start: 35 parts, among them IC1 STM32F042F6P6, IC2 MCP1700, IC3 TLV61225, J1 BATT, J2 MICROUSB, P1 SWD_TC, SW1 BOOTLOAD, SW2 PWR_SWITCH

Commit message: Version 1
Parts:
- removed D1, D2, D3, D4, D5, D6, D7, D8: LED, agg:0805-LED, symbol LED
- removed R10, R11, R5, R6, R8, R9: R, agg:0805, symbol R
- added D10, D13, D14, D3, D5, D6: LED_RABG, yule:CREE_RGB_LED, symbol LED_RABG
- added J3: CONN_01x08, yule:Interboard, symbol CONN_01x08
- added R12, R15, R17, R18, R20, R21, R23, R24, R26, R29, R32, R35, R36, R38, R39, R41, R42: 510, agg:0805, symbol R
- added SW3: BUTTON, yule:MOM_SWITCH, symbol SWITCH_MOM
- added X1: Silk_art, yule:tree_silk_scaled, symbol PART
- R4: value R -> 10k; Farnell (none) -> 9332391
- R7: value R -> 510; Digikey (none) -> Value; Farnell (none) -> 9333312; Fieldname (none) -> Value
- SW1: footprint agg:MOM_SWITCH -> yule:MOM_SWITCH; Digikey (none) -> Value; Fieldname (none) -> Value
Connections:
- net LED7 is gone; now on net BUTTON: IC1.13 (PA7)
- net 3v3: now also D10.2 (COMMON_ANODE), D13.2 (COMMON_ANODE), D14.2 (COMMON_ANODE), D3.2 (COMMON_ANODE), D5.2 (COMMON_ANODE), D6.2 (COMMON_ANODE), J3.4, J3.5, SW3.1 ("~")
- net GND: now also R4.2
- net LED1R: now reaches R7.2
- net LED1R: now also IC1.6 (PA0), J3.1, R17.2, R18.2
- net LED1 renamed BUTTON
- net BUTTON: now also SW3.2 ("~"); no longer IC1.6 (PA0)
- net LED2 renamed LED1G
- net LED1G: now also J3.2, R12.2, R20.2, R21.2
- net LED3 renamed LED1B
- net LED1B: now also J3.3, R15.2, R23.2, R24.2
- net LED4: no longer names the net of R7.1
- net LED4: now also D3.1 (RED_CATHODE); no longer IC1.9 (PA3)
- net LED5 renamed LED2G
- net LED2G: now also J3.8, R29.2, R38.2, R39.2
- net LED6 renamed LED2B
- net LED2B: now also J3.6, R32.2, R41.2, R42.2
- net LED8: no longer names the net of IC1.14 (PB1)
- new net: D3.3 (BLUE_CATHODE), R15.1
- new net: D3.4 (GREEN_CATHODE), R12.1
- new net: D5.1 (RED_CATHODE), R17.1
- new net: D5.3 (BLUE_CATHODE), R23.1
- new net: D5.4 (GREEN_CATHODE), R20.1
- new net: D6.1 (RED_CATHODE), R18.1
- new net: D6.3 (BLUE_CATHODE), R24.1
- new net: D6.4 (GREEN_CATHODE), R21.1
- new net: D10.1 (RED_CATHODE), R26.1
- new net: D10.3 (BLUE_CATHODE), R32.1
- new net: D10.4 (GREEN_CATHODE), R29.1
- new net: D13.1 (RED_CATHODE), R35.1
- new net: D13.3 (BLUE_CATHODE), R41.1
- new net: D13.4 (GREEN_CATHODE), R38.1
- new net: D14.1 (RED_CATHODE), R36.1
- new net: D14.3 (BLUE_CATHODE), R42.1
- new net: D14.4 (GREEN_CATHODE), R39.1
- new net LED2R: IC1.9 (PA3), J3.7, R26.2, R35.2, R36.2
- no-connect marks 7 -> 8
Other:
- note added: "E.g. for stepping through flashing speeds?"
- note removed: "Farnell LED codes:\n2099241 Red\n2099237 Orange\n2099242 Yellow\n2099235 Green\n2217980 Blue\n1716764 White"
- moved on the sheet: C1, C2, C3, C4, C5, C6, C7, IC1, IC2, IC3, J1, J2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
