File: pcb_2/tree_2.kicad_pcb (KiCad board)
At the start: 2 copper layers, 65 x 70 mm, 28 parts, among them J1 CONN_01x08, J2 CONN_01x08, X1 Silk_art, X2 Silk_art

Commit message: Fix circuit to account for LED currents: change resistor values, upgrade LDO regulator, use transistor array
Parts:
- R13, R14, R19, R22, R28, R30, R31, R33, R37, R40, R8, R9: value 510 -> 30
- R16, R25, R27, R34, R5, R6: value 510 -> 100
Changed lines of the file:
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@@
   )
   (setup
-    (last_trace_width 0.5)
+    (last_trace_width 0.25)
     (user_trace_width 0.15)
     (user_trace_width 0.2)
@@
       (drillshape 0)
       (scaleselection 1)
-      (outputdirectory ""))
+      (outputdirectory gerbers/))
   )
   (net 0 "")
@@
       (effects (font (size 1 1) (thickness 0.15)))
     )
-    (fp_text value 510 (at 2.425 0 90) (layer F.Fab)
+    (fp_text value 100 (at 2.425 0 90) (layer F.Fab)
       (effects (font (size 1 1) (thickness 0.15)))
     )
@@
       (effects (font (size 1 1) (thickness 0.15)))
     )
-    (fp_text value 510 (at 2.425 0 270) (layer F.Fab)
+    (fp_text value 100 (at 2.425 0 270) (layer F.Fab)
       (effects (font (size 1 1) (thickness 0.15)))
     )
@@
       (effects (font (size 1 1) (thickness 0.15)))
     )
-    (fp_text value 510 (at 2.425 0 90) (layer F.Fab)
+    (fp_text value 30 (at 2.425 0 90) (layer F.Fab)
       (effects (font (size 1 1) (thickness 0.15)))
     )
@@
       (effects (font (size 1 1) (thickness 0.15)))
     )
-    (fp_text value 510 (at 2.425 0 270) (layer F.Fab)
+    (fp_text value 30 (at 2.425 0 270) (layer F.Fab)
       (effects (font (size 1 1) (thickness 0.15)))
     )
@@
       (effects (font (size 1 1) (thickness 0.15)))
     )
-    (fp_text value 510 (at 2.425 0 90) (layer F.Fab)
+    (fp_text value 30 (at 2.425 0 90) (layer F.Fab)
       (effects (font (size 1 1) (thickness 0.15)))
     )
@@
       (effects (font (size 1 1) (thickness 0.15)))
     )
-    (fp_text value 510 (at 2.425 0 270) (layer F.Fab)
+    (fp_text value 30 (at 2.425 0 270) (layer F.Fab)
       (effects (font (size 1 1) (thickness 0.15)))
     )
@@
       (effects (font (size 1 1) (thickness 0.15)))
     )
-    (fp_text value 510 (at 2.425 0 90) (layer F.Fab)
+    (fp_text value 100 (at 2.425 0 90) (layer F.Fab)
       (effects (font (size 1 1) (thickness 0.15)))
     )
@@
       (effects (font (size 1 1) (thickness 0.15)))
     )
-    (fp_text value 510 (at 2.425 0 90) (layer F.Fab)
+    (fp_text value 30 (at 2.425 0 90) (layer F.Fab)
       (effects (font (size 1 1) (thickness 0.15)))
     )
@@
       (effects (font (size 1 1) (thickness 0.15)))
     )
-    (fp_text value 510 (at 2.425 0 90) (layer F.Fab)
+    (fp_text value 30 (at 2.425 0 90) (layer F.Fab)
       (effects (font (size 1 1) (thickness 0.15)))
     )
@@
       (effects (font (size 1 1) (thickness 0.15)))
     )
-    (fp_text value 510 (at 2.425 0 270) (layer F.Fab)
+    (fp_text value 100 (at 2.425 0 270) (layer F.Fab)
       (effects (font (size 1 1) (thickness 0.15)))
     )
@@
       (effects (font (size 1 1) (thickness 0.15)))
     )
-    (fp_text value 510 (at 2.425 0 90) (layer F.Fab)
+    (fp_text value 100 (at 2.425 0 90) (layer F.Fab)
       (effects (font (size 1 1) (thickness 0.15)))
     )
@@
       (effects (font (size 1 1) (thickness 0.15)))
     )
-    (fp_text value 510 (at 2.425 0 270) (layer F.Fab)
+    (fp_text value 30 (at 2.425 0 270) (layer F.Fab)
       (effects (font (size 1 1) (thickness 0.15)))
     )
@@
       (effects (font (size 1 1) (thickness 0.15)))
     )
-    (fp_text value 510 (at 2.425 0 90) (layer F.Fab)
+    (fp_text value 30 (at 2.425 0 90) (layer F.Fab)
       (effects (font (size 1 1) (thickness 0.15)))
     )
@@
       (effects (font (size 1 1) (thickness 0.15)))
     )
-    (fp_text value 510 (at 2.425 0 270) (layer F.Fab)
+    (fp_text value 30 (at 2.425 0 270) (layer F.Fab)
       (effects (font (size 1 1) (thickness 0.15)))
     )
@@
       (effects (font (size 1 1) (thickness 0.15)))
     )
-    (fp_text value 510 (at 2.425 0 90) (layer F.Fab)
+    (fp_text value 30 (at 2.425 0 90) (layer F.Fab)
       (effects (font (size 1 1) (thickness 0.15)))
     )
@@
       (effects (font (size 1 1) (thickness 0.15)))
     )
-    (fp_text value 510 (at 2.425 0 270) (layer F.Fab)
+    (fp_text value 100 (at 2.425 0 270) (layer F.Fab)
       (effects (font (size 1 1) (thickness 0.15)))
     )
@@
       (effects (font (size 1 1) (thickness 0.15)))
     )
-    (fp_text value 510 (at 2.425 0 270) (layer F.Fab)
+    (fp_text value 30 (at 2.425 0 270) (layer F.Fab)
       (effects (font (size 1 1) (thickness 0.15)))
     )
@@
       (effects (font (size 1 1) (thickness 0.15)))
     )
-    (fp_text value 510 (at 2.425 0 270) (layer F.Fab)
+    (fp_text value 30 (at 2.425 0 270) (layer F.Fab)
       (effects (font (size 1 1) (thickness 0.15)))
     )
@@
       (xy -10.888378 34.740037) (xy -10.440497 35.453794) (xy -10.274246 35.630556) (xy -10.051602 35.314088)) (layer B.SilkS) (width 0.01))
   )
+  (gr_arc (start 58 169) (end 59 169) (angle 90) (layer Edge.Cuts) (width 0.15))
   (gr_line (start 50 100) (end 70 100) (layer Edge.Cuts) (width 0.15))
-  (gr_arc (start 58 169) (end 59 169) (angle 90) (layer Edge.Cuts) (width 0.15))
   (gr_arc (start 62 154) (end 62 155) (angle 90) (layer Edge.Cuts) (width 0.15))
   (gr_line (start 61 130) (end 59 130) (layer Edge.Cuts) (width 0.15))
