File: pcb_2/tree_2.sch (KiCad schematic (older format))
At the start: 28 parts, among them J1 CONN_01x08, J2 CONN_01x08, X1 Silk_art, X2 Silk_art

Commit message: Tidy BOM
Parts:
- J1, J2, X1, X2: Farnell Value -> (none)
Changed lines of the file:
@@
 $EndComp
 $Comp
-L 3v3 #PWR3
+L 3v3 #PWR01
 U 1 1 58020594
 P 5550 2550
-F 0 "#PWR3" H 5550 2660 50  0001 L CNN
+F 0 "#PWR01" H 5550 2660 50  0001 L CNN
 F 1 "3v3" H 5550 2640 50  0000 C CNN
 F 2 "" H 5550 2550 60  0001 C CNN
@@
 $EndComp
 $Comp
-L 3v3 #PWR8
+L 3v3 #PWR02
 U 1 1 580205EC
 P 7350 2550
-F 0 "#PWR8" H 7350 2660 50  0001 L CNN
+F 0 "#PWR02" H 7350 2660 50  0001 L CNN
 F 1 "3v3" H 7350 2640 50  0000 C CNN
 F 2 "" H 7350 2550 60  0001 C CNN
@@
 $EndComp
 $Comp
-L 3v3 #PWR6
+L 3v3 #PWR03
 U 1 1 58020618
 P 6450 2550
-F 0 "#PWR6" H 6450 2660 50  0001 L CNN
+F 0 "#PWR03" H 6450 2660 50  0001 L CNN
 F 1 "3v3" H 6450 2640 50  0000 C CNN
 F 2 "" H 6450 2550 60  0001 C CNN
@@
 $EndComp
 $Comp
-L 3v3 #PWR7
+L 3v3 #PWR04
 U 1 1 5802011A
 P 7350 1100
-F 0 "#PWR7" H 7350 1210 50  0001 L CNN
+F 0 "#PWR04" H 7350 1210 50  0001 L CNN
 F 1 "3v3" H 7350 1190 50  0000 C CNN
 F 2 "" H 7350 1100 60  0001 C CNN
@@
 $EndComp
 $Comp
-L 3v3 #PWR4
+L 3v3 #PWR05
 U 1 1 5801F75B
 P 5600 1100
-F 0 "#PWR4" H 5600 1210 50  0001 L CNN
+F 0 "#PWR05" H 5600 1210 50  0001 L CNN
 F 1 "3v3" H 5600 1190 50  0000 C CNN
 F 2 "" H 5600 1100 60  0001 C CNN
@@
 $EndComp
 $Comp
-L 3v3 #PWR5
+L 3v3 #PWR06
 U 1 1 5801B866
 P 6450 1100
-F 0 "#PWR5" H 6450 1210 50  0001 L CNN
+F 0 "#PWR06" H 6450 1210 50  0001 L CNN
 F 1 "3v3" H 6450 1190 50  0000 C CNN
 F 2 "" H 6450 1100 60  0001 C CNN
@@
 F 2 "yule:Interboard" H 4000 1900 50  0001 C CNN
 F 3 "" H 4000 1900 50  0001 C CNN
-F 4 "Value" H 4000 1900 60  0001 C CNN "Farnell"
 	1    4000 1900
 	1    0    0    -1
@@
 F 2 "yule:Interboard" H 4000 2900 50  0001 C CNN
 F 3 "" H 4000 2900 50  0001 C CNN
-F 4 "Value" H 4000 2900 60  0001 C CNN "Farnell"
 	1    4000 2900
 	1    0    0    -1
@@
 Connection ~ 4600 2900
 $Comp
-L 3v3 #PWR1
+L 3v3 #PWR07
 U 1 1 5802A904
 P 4300 2250
-F 0 "#PWR1" H 4300 2360 50  0001 L CNN
+F 0 "#PWR07" H 4300 2360 50  0001 L CNN
 F 1 "3v3" H 4300 2340 50  0000 C CNN
 F 2 "" H 4300 2250 60  0001 C CNN
@@
 $EndComp
 $Comp
-L 3v3 #PWR2
+L 3v3 #PWR08
 U 1 1 5802A9EA
 P 4300 3250
-F 0 "#PWR2" H 4300 3360 50  0001 L CNN
+F 0 "#PWR08" H 4300 3360 50  0001 L CNN
 F 1 "3v3" H 4300 3340 50  0000 C CNN
 F 2 "" H 4300 3250 60  0001 C CNN
@@
 Connection ~ 4100 2250
 $Comp
-L PWR #FLG1
+L PWR #FLG09
 U 1 1 5802ABD2
 P 4200 2250
-F 0 "#FLG1" H 4200 2410 50  0001 C CNN
+F 0 "#FLG09" H 4200 2410 50  0001 C CNN
 F 1 "PWR" H 4200 2340 50  0000 C CNN
 F 2 "" H 4200 2250 50  0001 C CNN
@@
 F 2 "yule:tree_silk_scaled" H 8300 2350 50  0001 C CNN
 F 3 "" H 8300 2350 50  0001 C CNN
-F 4 "Value" H 8300 2350 60  0001 C CNN "Farnell"
 	1    8300 2350
 	1    0    0    -1
@@
 F 2 "yule:tree_silk_scaled" H 8300 2700 50  0001 C CNN
 F 3 "" H 8300 2700 50  0001 C CNN
-F 4 "Value" H 8300 2700 60  0001 C CNN "Farnell"
 	1    8300 2700
 	1    0    0    -1
